File: Hardware/Analog_Audio.kicad_sch (KiCad schematic)
At the start: 0 parts

Commit message: Major Updates to Schematic
Parts:
- added C6: 0.015u, symbol Device:C
- added C7: 0.1u, symbol Device:C
- added MK1: Microphone, Connector_PinHeader_2.54mm:PinHeader_1x02_P2.54mm_Vertical, symbol Device:Microphone
- added Q1: S8550, Package_TO_SOT_THT:TO-92_Inline, symbol Transistor_BJT:S8550
- added R10: 1K, symbol Device:R
- added R11, R8, R9: 10K, symbol Device:R
- added R12: 47K, symbol Device:R
- added R7: Photoresistor, OptoDevice:R_LDR_5.1x4.3mm_P3.4mm_Vertical, symbol Device:R_Photo
- added RV1: 50K, Potentiometer_SMD:Potentiometer_Bourns_3314J_Vertical, symbol Device:R_Potentiometer
Connections:
- new net: R12.1, RV1.3
- new net: C7.2, Q1.2 (B), R12.2
- new net: C6.2, MK1.2 (+), R10.1, R9.2
- new net: C7.1, R10.2
- new net +3V3: Q1.1 (E), R7.1, R9.1
- new net GND: C6.1, MK1.1 (-), R11.2, R8.1
- new net GPIO 34: R7.2, R8.2
- new net GPIO 35: Q1.3 (C), R11.1, RV1.2
- no-connect marks 0 -> 1
Other:
- note added: "Microphone"
- note added: "Photoresistor"

Commit message: Schematic V0.9 is complete
Parts:
- C6: footprint (none) -> Capacitor_THT:C_Disc_D4.3mm_W1.9mm_P5.00mm
- C7: footprint (none) -> Capacitor_SMD:C_0805_2012Metric
- R10, R11, R12, R8, R9: footprint (none) -> Resistor_SMD:R_0805_2012Metric
Changed lines of the file:
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@@
 			)
 		)
-		(property "Footprint" ""
+		(property "Footprint" "Resistor_SMD:R_0805_2012Metric"
 			(at 167.132 125.73 90)
 			(hide yes)
@@
 			)
 		)
-		(property "Footprint" ""
+		(property "Footprint" "Resistor_SMD:R_0805_2012Metric"
 			(at 86.36 113.538 90)
 			(hide yes)
@@
 			)
 		)
-		(property "Footprint" ""
+		(property "Footprint" "Resistor_SMD:R_0805_2012Metric"
 			(at 158.242 110.49 90)
 			(hide yes)
@@
 			)
 		)
-		(property "Footprint" ""
+		(property "Footprint" "Capacitor_THT:C_Disc_D4.3mm_W1.9mm_P5.00mm"
 			(at 140.6652 104.14 0)
 			(hide yes)
@@
 			)
 		)
-		(property "Footprint" ""
+		(property "Footprint" "Capacitor_SMD:C_0805_2012Metric"
 			(at 160.9852 125.73 0)
 			(hide yes)
@@
 			)
 		)
-		(property "Footprint" ""
+		(property "Footprint" "Resistor_SMD:R_0805_2012Metric"
 			(at 158.242 87.63 90)
 			(hide yes)
@@
 			)
 		)
-		(property "Footprint" ""
+		(property "Footprint" "Resistor_SMD:R_0805_2012Metric"
 			(at 193.04 121.158 90)
 			(hide yes)
