File: Hardware/Digital_Bus.kicad_sch (KiCad schematic)
At the start: 0 parts

Commit message: Major Updates to Schematic
Parts:
- added C10, C8: 10u, symbol Device:C
- added C11, C9: 0.1u, symbol Device:C
- added C2, C3: 0.1uF, symbol Device:C
- added J3: DM3D-SF, Micro_SD_Card:HRS_DM3D-SF, symbol DM3D-SF:DM3D-SF
- added R14: 10K, symbol Device:R
- added R5, R6: 4.7K, symbol Device:R
- added U1: BME280, Package_LGA:Bosch_LGA-8_2.5x2.5mm_P0.65mm_ClockwisePinNumbering, symbol Sensor:BME280
- added U3: ENS160-BGLT, Custom_Sensors:XDCR_ENS160-BGLT, symbol ENS160-BGLT:ENS160-BGLT
Connections:
- net +3V3: now also C10.1, C11.1, C2.1, C3.1, C9.1, J3.4 (VDD), R14.1, R5.2, R6.2, U1.2 (CSB), U1.6 (VDDIO), U1.8 (VDD), U3.5 (VDDIO), U3.7 (~{CS})
- net GND: now also C10.2, C11.2, C2.2, C3.2, C8.1, C9.2, J3.6 (VSS), J3.S1 (SHIELD), J3.S2 (SHIELD__1), J3.S3 (SHIELD__2), J3.S4 (SHIELD__3), U1.1 (GND), U1.5 (SDO), U1.7 (GND), U3.3 (MISO/ADDR), U3.8 (VSS), U3.9 (VSS__1)
- new net 1.8V: C8.2, U3.4 (VDD)
- new net MISO: J3.7 (DAT0)
- new net MOSI: J3.3 (CMD)
- new net SCK: J3.5 (CLK)
- new net SCL: R6.1, U1.4 (SCK), U3.2 (SCLK/SCL)
- new net SDA: R5.1, U1.3 (SDI), U3.1 (MOSI/SDA)
- new net SD_CS: J3.2 (CD/DAT3), R14.2
- no-connect marks 0 -> 5
Other:
- note added: "Air Quality Sensor"
- note added: "SD Card"
- note added: "Temperature/Humidity/Pressure"

Commit message: Schematic V0.9 is complete
Parts:
- C10, C11, C8, C9: footprint (none) -> Capacitor_SMD:C_0805_2012Metric
- C2, C3: value 0.1uF -> 0.1u; footprint (none) -> Capacitor_SMD:C_0805_2012Metric
- R14, R5, R6: footprint (none) -> Resistor_SMD:R_0805_2012Metric
Changed lines of the file:
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@@
 	)
 	(junction
+		(at 157.48 41.91)
+		(diameter 0)
+		(color 0 0 0 0)
+	)
+	(junction
 		(at 107.95 142.24)
 		(diameter 0)
@@
 	)
 	(junction
-		(at 160.02 74.93)
+		(at 157.48 74.93)
 		(diameter 0)
 		(color 0 0 0 0)
@@
 	)
 	(junction
+		(at 160.02 74.93)
+		(diameter 0)
+		(color 0 0 0 0)
+	)
+	(junction
 		(at 160.02 69.85)
 		(diameter 0)
@@
 	(wire
 		(pts
-			(xy 160.02 74.93) (xy 160.02 76.2)
+			(xy 157.48 74.93) (xy 160.02 74.93)
+		)
+		(stroke
+			(width 0)
+			(type default)
+		)
+	)
+	(wire
+		(pts
+			(xy 165.1 74.93) (xy 165.1 76.2)
 		)
 		(stroke
@@
 	(wire
 		(pts
-			(xy 156.21 74.93) (xy 160.02 74.93)
+			(xy 156.21 74.93) (xy 157.48 74.93)
 		)
 		(stroke
@@
 	(wire
 		(pts
-			(xy 156.21 41.91) (xy 161.29 41.91)
+			(xy 156.21 41.91) (xy 157.48 41.91)
 		)
 		(stroke
@@
 	(wire
 		(pts
+			(xy 157.48 41.91) (xy 161.29 41.91)
+		)
+		(stroke
+			(width 0)
+			(type default)
+		)
+	)
+	(wire
+		(pts
 			(xy 153.67 138.43) (xy 153.67 139.7)
 		)
@@
 	(wire
 		(pts
+			(xy 165.1 74.93) (xy 160.02 74.93)
+		)
+		(stroke
+			(width 0)
+			(type default)
+		)
+	)
+	(wire
+		(pts
 			(xy 67.31 148.59) (xy 67.31 152.4)
 		)
@@
 	(symbol
 		(lib_id "power:GND")
-		(at 160.02 76.2 0)
+		(at 165.1 76.2 0)
 		(unit 1)
 		(body_style 1)
@@
 		(fields_autoplaced yes)
 		(property "Reference" "#PWR029"
-			(at 160.02 82.55 0)
+			(at 165.1 82.55 0)
 			(hide yes)
 			(show_name no)
@@
 		)
 		(property "Value" "GND"
-			(at 160.02 81.28 0)
+			(at 165.1 81.28 0)
 			(show_name no)
 			(do_not_autoplace no)
@@
 		)
 		(property "Footprint" ""
-			(at 160.02 76.2 0)
+			(at 165.1 76.2 0)
 			(hide yes)
 			(show_name no)
@@
 		)
 		(property "Datasheet" ""
-			(at 160.02 76.2 0)
+			(at 165.1 76.2 0)
 			(hide yes)
 			(show_name no)
@@
 		)
 		(property "Description" "Power symbol creates a global label with name \"GND\" , ground"
-			(at 160.02 76.2 0)
+			(at 165.1 76.2 0)
 			(hide yes)
 			(show_name no)
@@
 			)
 		)
-		(property "Footprint" ""
+		(property "Footprint" "Resistor_SMD:R_0805_2012Metric"
 			(at 103.632 50.8 90)
 			(hide yes)
@@
 			)
 		)
-		(property "Footprint" ""
+		(property "Footprint" "Capacitor_SMD:C_0805_2012Metric"
 			(at 206.7052 129.54 0)
 			(hide yes)
@@
 	)
 	(symbol
+		(lib_id "power:PWR_FLAG")
+		(at 157.48 74.93 180)
+		(unit 1)
+		(body_style 1)
+		(exclude_from_sim no)
+		(in_bom yes)
+		(on_board yes)
+		(in_pos_files yes)
+		(dnp no)
+		(fields_autoplaced yes)
+		(property "Reference" "#FLG02"
+			(at 157.48 76.835 0)
+			(hide yes)
+			(show_name no)
+			(do_not_autoplace no)
+			(effects
+				(font
+					(size 1.27 1.27)
+				)
+			)
+		)
+		(property "Value" "PWR_FLAG"
+			(at 157.48 80.01 0)
+			(show_name no)
+			(do_not_autoplace no)
+			(effects
+				(font
+					(size 1.27 1.27)
+				)
+			)
+		)
+		(property "Footprint" ""
+			(at 157.48 74.93 0)
+			(hide yes)
+			(show_name no)
+			(do_not_autoplace no)
+			(effects
+				(font
+					(size 1.27 1.27)
+				)
+			)
+		)
+		(property "Datasheet" ""
+			(at 157.48 74.93 0)
+			(hide yes)
+			(show_name no)
+			(do_not_autoplace no)
+			(effects
+				(font
+					(size 1.27 1.27)
+				)
+			)
+		)
+		(property "Description" "Special symbol for telling ERC where power comes from"
+			(at 157.48 74.93 0)
+			(hide yes)
+			(show_name no)
+			(do_not_autoplace no)
+			(effects
+				(font
+					(size 1.27 1.27)
+				)
+			)
+		)
+		(pin "1"
+		)
+		(instances
+			(project "ESP32_IOT_PCB"
+				(path "/22b198a3-add8-435b-b36e-05e6b8d693ec/1ac80ee3-fd26-42f2-b2cb-8a8f62615b81"
+					(reference "#FLG02")
+					(unit 1)
+				)
+			)
+		)
+	)
+	(symbol
+		(lib_id "power:PWR_FLAG")
+		(at 157.48 41.91 180)
+		(unit 1)
+		(body_style 1)
+		(exclude_from_sim no)
+		(in_bom yes)
+		(on_board yes)
+		(in_pos_files yes)
+		(dnp no)
+		(fields_autoplaced yes)
+		(property "Reference" "#FLG01"
+			(at 157.48 43.815 0)
+			(hide yes)
+			(show_name no)
+			(do_not_autoplace no)
+			(effects
+				(font
+					(size 1.27 1.27)
+				)
+			)
+		)
+		(property "Value" "PWR_FLAG"
+			(at 157.48 46.99 0)
+			(show_name no)
+			(do_not_autoplace no)
+			(effects
+				(font
+					(size 1.27 1.27)
+				)
+			)
+		)
+		(property "Footprint" ""
+			(at 157.48 41.91 0)
+			(hide yes)
+			(show_name no)
+			(do_not_autoplace no)
+			(effects
+				(font
+					(size 1.27 1.27)
+				)
+			)
+		)
+		(property "Datasheet" ""
+			(at 157.48 41.91 0)
+			(hide yes)
+			(show_name no)
+			(do_not_autoplace no)
+			(effects
+				(font
+					(size 1.27 1.27)
+				)
+			)
+		)
+		(property "Description" "Special symbol for telling ERC where power comes from"
+			(at 157.48 41.91 0)
+			(hide yes)
+			(show_name no)
+			(do_not_autoplace no)
+			(effects
+				(font
+					(size 1.27 1.27)
+				)
+			)
+		)
+		(pin "1"
+		)
+		(instances
+			(project "ESP32_IOT_PCB"
+				(path "/22b198a3-add8-435b-b36e-05e6b8d693ec/1ac80ee3-fd26-42f2-b2cb-8a8f62615b81"
+					(reference "#FLG01")
+					(unit 1)
+				)
+			)
+		)
+	)
+	(symbol
 		(lib_id "power:+3V3")
 		(at 153.67 138.43 0)
@@
 			)
 		)
-		(property "Footprint" ""
+		(property "Footprint" "Resistor_SMD:R_0805_2012Metric"
 			(at 106.172 135.89 90)
 			(hide yes)
@@
 			)
 		)
-		(property "Footprint" ""
+		(property "Footprint" "Capacitor_SMD:C_0805_2012Metric"
 			(at 164.7952 53.34 0)
 			(hide yes)
@@
 			)
 		)
-		(property "Value" "0.1uF"
+		(property "Value" "0.1u"
 			(at 55.88 109.22 90)
 			(show_name no)
@@
 			)
 		)
-		(property "Footprint" ""
+		(property "Footprint" "Capacitor_SMD:C_0805_2012Metric"
 			(at 52.07 115.2652 0)
 			(hide yes)
@@
 			)
 		)
-		(property "Footprint" ""
+		(property "Footprint" "Resistor_SMD:R_0805_2012Metric"
 			(at 85.852 137.16 90)
 			(hide yes)
@@
 			)
 		)
-		(property "Footprint" ""
+		(property "Footprint" "Capacitor_SMD:C_0805_2012Metric"
 			(at 214.3252 144.78 0)
 			(hide yes)
@@
 			)
 		)
-		(property "Footprint" ""
+		(property "Footprint" "Capacitor_SMD:C_0805_2012Metric"
 			(at 176.2252 53.34 0)
 			(hide yes)
@@
 			)
 		)
-		(property "Value" "0.1uF"
+		(property "Value" "0.1u"
 			(at 81.28 109.22 90)
 			(show_name no)
@@
 			)
 		)
-		(property "Footprint" ""
+		(property "Footprint" "Capacitor_SMD:C_0805_2012Metric"
 			(at 85.09 113.3348 0)
 			(hide yes)
